File: hdw/Incrementor/Clock_Output.kicad_sch (KiCad schematic)
At the start: 7 parts, among them J1901 CLK_OUT, U1901 74LVC1G17

Commit message: renamed project, removed stuff I dont need
Other:
- title: Incrementor -> Stopwatch
Changed lines of the file:
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@@
   (paper "A")
   (title_block
-    (title "Incrementor")
-    (date "2019-09-03")
+    (title "Stopwatch")
+    (date "2024-01-02")
     (rev "A")
     (company "Drew Maatman")
