File: hdw/Incrementor/Oscillator.kicad_sch (KiCad schematic)
At the start: 12 parts, among them U401 CD4024, U402 CD4040, X401 ECS-327KE

Commit message: renamed project, removed stuff I dont need
Other:
- title: Incrementor -> Stopwatch
Changed lines of the file:
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@@
   (paper "A")
   (title_block
-    (title "Incrementor")
-    (date "2019-09-03")
+    (title "Stopwatch")
+    (date "2024-01-02")
     (rev "A")
     (company "Drew Maatman")
@@
     )
     (pin "1")
+    (instances
+      (project "Stopwatch"
+        (path "/c0d2575b-aec2-49ed-8c32-97fe6e68824c/00000000-0000-0000-0000-00005d784813"
+          (reference "#PWR0402") (unit 1)
+        )
+      )
+    )
   )
   (symbol (lib_id "74xx:74HC4024") (at 137.414 86.614 0) (unit 1)
@@
     (pin "9")
     (instances
-      (project "Incrementor"
+      (project "Stopwatch"
         (path "/c0d2575b-aec2-49ed-8c32-97fe6e68824c/00000000-0000-0000-0000-00005d784813"
           (reference "U401") (unit 1)
@@
     (pin "2")
     (instances
-      (project "Incrementor"
+      (project "Stopwatch"
         (path "/c0d2575b-aec2-49ed-8c32-97fe6e68824c/00000000-0000-0000-0000-00005d784813"
           (reference "C401") (unit 1)
@@
     (pin "2")
     (instances
-      (project "Incrementor"
+      (project "Stopwatch"
         (path "/c0d2575b-aec2-49ed-8c32-97fe6e68824c/00000000-0000-0000-0000-00005d784813"
           (reference "C402") (unit 1)
@@
     (pin "2")
     (instances
-      (project "Incrementor"
+      (project "Stopwatch"
         (path "/c0d2575b-aec2-49ed-8c32-97fe6e68824c/00000000-0000-0000-0000-00005d784813"
           (reference "C403") (unit 1)
@@
     )
     (pin "1")
+    (instances
+      (project "Stopwatch"
+        (path "/c0d2575b-aec2-49ed-8c32-97fe6e68824c/00000000-0000-0000-0000-00005d784813"
+          (reference "#PWR0403") (unit 1)
+        )
+      )
+    )
   )
   (symbol (lib_id "power:GND") (at 42.418 122.936 0) (unit 1)
@@
     )
     (pin "1")
+    (instances
+      (project "Stopwatch"
+        (path "/c0d2575b-aec2-49ed-8c32-97fe6e68824c/00000000-0000-0000-0000-00005d784813"
+          (reference "#PWR0404") (unit 1)
+        )
+      )
+    )
   )
   (symbol (lib_id "Custom_Library:R_Custom") (at 98.298 97.536 0) (unit 1)
@@
     (pin "2")
     (instances
-      (project "Incrementor"
+      (project "Stopwatch"
         (path "/c0d2575b-aec2-49ed-8c32-97fe6e68824c/00000000-0000-0000-0000-00005d784813"
           (reference "R401") (unit 1)
@@
     (pin "1")
     (instances
-      (project "Incrementor"
+      (project "Stopwatch"
         (path "/c0d2575b-aec2-49ed-8c32-97fe6e68824c/00000000-0000-0000-0000-00005d784813"
           (reference "#PWR0405") (unit 1)
@@
     )
     (pin "1")
+    (instances
+      (project "Stopwatch"
+        (path "/c0d2575b-aec2-49ed-8c32-97fe6e68824c/00000000-0000-0000-0000-00005d784813"
+          (reference "#PWR0407") (unit 1)
+        )
+      )
+    )
   )
   (symbol (lib_id "power:GND") (at 137.414 99.314 0) (unit 1)
@@
     )
     (pin "1")
+    (instances
+      (project "Stopwatch"
+        (path "/c0d2575b-aec2-49ed-8c32-97fe6e68824c/00000000-0000-0000-0000-00005d784813"
+          (reference "#PWR0408") (unit 1)
+        )
+      )
+    )
   )
   (symbol (lib_id "power:GND") (at 115.062 101.346 0) (unit 1)
@@
     (pin "1")
     (instances
-      (project "Incrementor"
+      (project "Stopwatch"
         (path "/c0d2575b-aec2-49ed-8c32-97fe6e68824c/00000000-0000-0000-0000-00005d784813"
           (reference "#PWR0406") (unit 1)
@@
     (pin "2")
     (instances
-      (project "Incrementor"
+      (project "Stopwatch"
         (path "/c0d2575b-aec2-49ed-8c32-97fe6e68824c/00000000-0000-0000-0000-00005d784813"
           (reference "R402") (unit 1)
@@
     (pin "2")
     (instances
-      (project "Incrementor"
+      (project "Stopwatch"
         (path "/c0d2575b-aec2-49ed-8c32-97fe6e68824c/00000000-0000-0000-0000-00005d784813"
           (reference "C404") (unit 1)
@@
     )
     (pin "1")
+    (instances
+      (project "Stopwatch"
+        (path "/c0d2575b-aec2-49ed-8c32-97fe6e68824c/00000000-0000-0000-0000-00005d784813"
+          (reference "#PWR0410") (unit 1)
+        )
+      )
+    )
   )
   (symbol (lib_id "4xxx:4040") (at 225.044 92.964 0) (unit 1)
@@
     (pin "9")
     (instances
-      (project "Incrementor"
+      (project "Stopwatch"
         (path "/c0d2575b-aec2-49ed-8c32-97fe6e68824c/00000000-0000-0000-0000-00005d784813"
           (reference "U402") (unit 1)
@@
     )
     (pin "1")
+    (instances
+      (project "Stopwatch"
+        (path "/c0d2575b-aec2-49ed-8c32-97fe6e68824c/00000000-0000-0000-0000-00005d784813"
+          (reference "#PWR0414") (unit 1)
+        )
+      )
+    )
   )
   (symbol (lib_id "Incrementor-rescue:+3.3V-power") (at 225.044 72.644 0) (unit 1)
@@
     )
     (pin "1")
+    (instances
+      (project "Stopwatch"
+        (path "/c0d2575b-aec2-49ed-8c32-97fe6e68824c/00000000-0000-0000-0000-00005d784813"
+          (reference "#PWR0413") (unit 1)
+        )
+      )
+    )
   )
   (symbol (lib_id "Custom_Library:R_Custom") (at 200.152 96.266 0) (unit 1)
@@
     (pin "2")
     (instances
-      (project "Incrementor"
+      (project "Stopwatch"
         (path "/c0d2575b-aec2-49ed-8c32-97fe6e68824c/00000000-0000-0000-0000-00005d784813"
           (reference "R404") (unit 1)
@@
     (pin "1")
     (instances
-      (project "Incrementor"
+      (project "Stopwatch"
         (path "/c0d2575b-aec2-49ed-8c32-97fe6e68824c/00000000-0000-0000-0000-00005d784813"
           (reference "#PWR0412") (unit 1)
@@
     (pin "2")
     (instances
-      (project "Incrementor"
+      (project "Stopwatch"
         (path "/c0d2575b-aec2-49ed-8c32-97fe6e68824c/00000000-0000-0000-0000-00005d784813"
           (reference "R403") (unit 1)
@@
     (pin "1")
     (instances
-      (project "Incrementor"
+      (project "Stopwatch"
         (path "/c0d2575b-aec2-49ed-8c32-97fe6e68824c/00000000-0000-0000-0000-00005d784813"
           (reference "#PWR0411") (unit 1)
@@
     (pin "2")
     (instances
-      (project "Incrementor"
+      (project "Stopwatch"
         (path "/c0d2575b-aec2-49ed-8c32-97fe6e68824c/00000000-0000-0000-0000-00005d784813"
           (reference "C407") (unit 1)
@@
     )
     (pin "1")
+    (instances
+      (project "Stopwatch"
+        (path "/c0d2575b-aec2-49ed-8c32-97fe6e68824c/00000000-0000-0000-0000-00005d784813"
+          (reference "#PWR0415") (unit 1)
+        )
+      )
+    )
   )
   (symbol (lib_id "power:GND") (at 225.044 135.636 0) (unit 1)
@@
     )
     (pin "1")
+    (instances
+      (project "Stopwatch"
+        (path "/c0d2575b-aec2-49ed-8c32-97fe6e68824c/00000000-0000-0000-0000-00005d784813"
+          (reference "#PWR0416") (unit 1)
+        )
+      )
+    )
   )
   (symbol (lib_id "Incrementor-rescue:+3.3V-power") (at 137.16 109.728 0) (unit 1)
@@
     )
     (pin "1")
+    (instances
+      (project "Stopwatch"
+        (path "/c0d2575b-aec2-49ed-8c32-97fe6e68824c/00000000-0000-0000-0000-00005d784813"
+          (reference "#PWR0409") (unit 1)
+        )
+      )
+    )
   )
   (symbol (lib_id "Incrementor-rescue:+3.3V-power") (at 42.672 80.518 0) (unit 1)
@@
     )
     (pin "1")
+    (instances
+      (project "Stopwatch"
+        (path "/c0d2575b-aec2-49ed-8c32-97fe6e68824c/00000000-0000-0000-0000-00005d784813"
+          (reference "#PWR?") (unit 1)
+        )
+      )
+    )
   )
   (symbol (lib_id "Incrementor-rescue:+3.3V-power") (at 33.02 86.106 0) (unit 1)
@@
     )
     (pin "1")
+    (instances
+      (project "Stopwatch"
+        (path "/c0d2575b-aec2-49ed-8c32-97fe6e68824c/00000000-0000-0000-0000-00005d784813"
+          (reference "#PWR?") (unit 1)
+        )
+      )
+    )
   )
   (symbol (lib_id "Custom_Library:ECS-327KE") (at 42.672 88.138 0) (unit 1)
@@
     (pin "4")
     (instances
-      (project "Incrementor"
+      (project "Stopwatch"
         (path "/c0d2575b-aec2-49ed-8c32-97fe6e68824c/00000000-0000-0000-0000-00005d784813"
           (reference "X401") (unit 1)
