File: hdw/Incrementor/POS12_Power_Input.kicad_sch (KiCad schematic)
At the start: 19 parts, among them J201 +12V IN, U201 TPS26600RHFT

Commit message: renamed project, removed stuff I dont need
Connections:
- net at U201.12 (OVP): now also R?.1, R?.2
Other:
- title: Incrementor -> Stopwatch
Changed lines of the file:
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@@
   (paper "A")
   (title_block
-    (title "Incrementor")
-    (date "2019-09-03")
+    (title "Stopwatch")
+    (date "2024-01-02")
     (rev "A")
     (company "Drew Maatman")
@@
   (symbol (lib_id "Custom_Library:C_Custom") (at 134.62 155.194 0) (unit 1)
     (in_bom yes) (on_board yes) (dnp no)
-    (property "Reference" "C?" (at 135.255 152.654 0)
+    (property "Reference" "C201" (at 135.255 152.654 0)
       (effects (font (size 1.27 1.27)) (justify left))
     )
@@
     (pin "2")
     (instances
-      (project "Incrementor"
+      (project "Stopwatch"
         (path "/c0d2575b-aec2-49ed-8c32-97fe6e68824c/00000000-0000-0000-0000-00005d77a516"
           (reference "C201") (unit 1)
@@
   (symbol (lib_id "Custom_Library:C_Custom") (at 142.24 155.194 0) (unit 1)
     (in_bom yes) (on_board yes) (dnp no)
-    (property "Reference" "C?" (at 142.875 152.654 0)
+    (property "Reference" "C202" (at 142.875 152.654 0)
       (effects (font (size 1.27 1.27)) (justify left))
     )
@@
     (pin "2")
     (instances
-      (project "Incrementor"
+      (project "Stopwatch"
         (path "/c0d2575b-aec2-49ed-8c32-97fe6e68824c/00000000-0000-0000-0000-00005d77a516"
           (reference "C202") (unit 1)
@@
   (symbol (lib_id "Custom_Library:C_Custom") (at 149.86 155.194 0) (unit 1)
     (in_bom yes) (on_board yes) (dnp no)
-    (property "Reference" "C?" (at 150.495 152.654 0)
+    (property "Reference" "C203" (at 150.495 152.654 0)
       (effects (font (size 1.27 1.27)) (justify left))
     )
@@
     (pin "2")
     (instances
-      (project "Incrementor"
+      (project "Stopwatch"
         (path "/c0d2575b-aec2-49ed-8c32-97fe6e68824c/00000000-0000-0000-0000-00005d77a516"
           (reference "C203") (unit 1)
@@
     )
     (pin "1")
+    (instances
+      (project "Stopwatch"
+        (path "/c0d2575b-aec2-49ed-8c32-97fe6e68824c/00000000-0000-0000-0000-00005d77a516"
+          (reference "#PWR0208") (unit 1)
+        )
+      )
+    )
   )
   (symbol (lib_id "Custom_Library:+12Vin") (at 83.82 54.864 0) (unit 1)
@@
     )
     (pin "1")
+    (instances
+      (project "Stopwatch"
+        (path "/c0d2575b-aec2-49ed-8c32-97fe6e68824c/00000000-0000-0000-0000-00005d77a516"
+          (reference "#PWR0204") (unit 1)
+        )
+      )
+    )
   )
   (symbol (lib_id "Custom_Library:+12Vin") (at 142.24 149.352 0) (unit 1)
@@
     )
     (pin "1")
+    (instances
+      (project "Stopwatch"
+        (path "/c0d2575b-aec2-49ed-8c32-97fe6e68824c/00000000-0000-0000-0000-00005d77a516"
+          (reference "#PWR0207") (unit 1)
+        )
+      )
+    )
   )
   (symbol (lib_id "Custom_Library:CP_Tant_Custom") (at 214.122 62.738 0) (unit 1)
@@
     (pin "2")
     (instances
-      (project "Incrementor"
+      (project "Stopwatch"
         (path "/c0d2575b-aec2-49ed-8c32-97fe6e68824c/00000000-0000-0000-0000-00005d77a516"
           (reference "C205") (unit 1)
@@
     )
     (pin "1")
+    (instances
+      (project "Stopwatch"
+        (path "/c0d2575b-aec2-49ed-8c32-97fe6e68824c/00000000-0000-0000-0000-00005d77a516"
+          (reference "#PWR0212") (unit 1)
+        )
+      )
+    )
   )
   (symbol (lib_id "power:+12V") (at 214.122 54.864 0) (unit 1)
@@
     )
     (pin "1")
+    (instances
+      (project "Stopwatch"
+        (path "/c0d2575b-aec2-49ed-8c32-97fe6e68824c/00000000-0000-0000-0000-00005d77a516"
+          (reference "#PWR0211") (unit 1)
+        )
+      )
+    )
   )
   (symbol (lib_id "power:PWR_FLAG") (at 195.072 55.118 0) (unit 1)
@@
     (pin "1")
     (instances
-      (project "Incrementor"
+      (project "Stopwatch"
         (path "/c0d2575b-aec2-49ed-8c32-97fe6e68824c/00000000-0000-0000-0000-00005d77a516"
           (reference "#FLG0203") (unit 1)
@@
     )
     (pin "1")
+    (instances
+      (project "Stopwatch"
+        (path "/c0d2575b-aec2-49ed-8c32-97fe6e68824c/00000000-0000-0000-0000-00005d77a516"
+          (reference "#PWR0202") (unit 1)
+        )
+      )
+    )
   )
   (symbol (lib_id "power:PWR_FLAG") (at 51.562 103.378 0) (unit 1)
@@
     (pin "1")
     (instances
-      (project "Incrementor"
+      (project "Stopwatch"
         (path "/c0d2575b-aec2-49ed-8c32-97fe6e68824c/00000000-0000-0000-0000-00005d77a516"
           (reference "#FLG0201") (unit 1)
@@
     (pin "1")
     (instances
-      (project "Incrementor"
+      (project "Stopwatch"
         (path "/c0d2575b-aec2-49ed-8c32-97fe6e68824c/00000000-0000-0000-0000-00005d77a516"
           (reference "#FLG0202") (unit 1)
@@
     (pin "2")
     (instances
-      (project "Incrementor"
+      (project "Stopwatch"
         (path "/c0d2575b-aec2-49ed-8c32-97fe6e68824c/00000000-0000-0000-0000-00005d77a516"
           (reference "D201") (unit 1)
@@
     )
     (pin "1")
+    (instances
+      (project "Stopwatch"
+        (path "/c0d2575b-aec2-49ed-8c32-97fe6e68824c/00000000-0000-0000-0000-00005d77a516"
+          (reference "#PWR0205") (unit 1)
+        )
+      )
+    )
   )
   (symbol (lib_id "Connector:Barrel_Jack_Switch") (at 40.132 59.436 0) (unit 1)
@@
     (pin "3")
     (instances
-      (project "Incrementor"
+      (project "Stopwatch"
         (path "/c0d2575b-aec2-49ed-8c32-97fe6e68824c/00000000-0000-0000-0000-00005d77a516"
           (reference "J201") (unit 1)
@@
     )
     (pin "1")
+    (instances
+      (project "Stopwatch"
+        (path "/c0d2575b-aec2-49ed-8c32-97fe6e68824c/00000000-0000-0000-0000-00005d77a516"
+          (reference "#PWR0201") (unit 1)
+        )
+      )
+    )
   )
   (symbol (lib_id "Incrementor-rescue:TPS26600RHFT-Custom_Library") (at 142.24 92.456 0) (unit 1)
@@
     (pin "9")
     (instances
-      (project "Incrementor"
+      (project "Stopwatch"
         (path "/c0d2575b-aec2-49ed-8c32-97fe6e68824c"
           (reference "U201") (unit 1)
@@
     )
     (pin "1")
+    (instances
+      (project "Stopwatch"
+        (path "/c0d2575b-aec2-49ed-8c32-97fe6e68824c/00000000-0000-0000-0000-00005d77a516"
+          (reference "#PWR0206") (unit 1)
+        )
+      )
+    )
   )
   (symbol (lib_id "Custom_Library:R_Custom") (at 167.894 97.282 0) (unit 1)
@@
     (pin "2")
     (instances
-      (project "Incrementor"
+      (project "Stopwatch"
         (path "/c0d2575b-aec2-49ed-8c32-97fe6e68824c/00000000-0000-0000-0000-00005d6c0d23"
           (reference "R?") (unit 1)
@@
     )
     (pin "1")
+    (instances
+      (project "Stopwatch"
+        (path "/c0d2575b-aec2-49ed-8c32-97fe6e68824c/00000000-0000-0000-0000-00005d77a516"
+          (reference "#PWR0209") (unit 1)
+        )
+      )
+    )
   )
   (symbol (lib_id "Custom_Library:R_Custom") (at 166.116 132.334 0) (unit 1)
@@
     (pin "2")
     (instances
-      (project "Incrementor"
+      (project "Stopwatch"
         (path "/c0d2575b-aec2-49ed-8c32-97fe6e68824c/00000000-0000-0000-0000-00005d6c0d23"
           (reference "R?") (unit 1)
@@
     (pin "2")
     (instances
-      (project "Incrementor"
+      (project "Stopwatch"
         (path "/c0d2575b-aec2-49ed-8c32-97fe6e68824c/00000000-0000-0000-0000-00005d6c0d23"
           (reference "R?") (unit 1)
@@
     (pin "2")
     (instances
-      (project "Incrementor"
+      (project "Stopwatch"
         (path "/c0d2575b-aec2-49ed-8c32-97fe6e68824c/00000000-0000-0000-0000-00005d6c0d23"
           (reference "R?") (unit 1)
@@
     (pin "2")
     (instances
-      (project "Incrementor"
+      (project "Stopwatch"
         (path "/c0d2575b-aec2-49ed-8c32-97fe6e68824c/00000000-0000-0000-0000-00005d6c0d23"
           (reference "R?") (unit 1)
@@
     (pin "2")
     (instances
-      (project "Incrementor"
+      (project "Stopwatch"
         (path "/c0d2575b-aec2-49ed-8c32-97fe6e68824c/00000000-0000-0000-0000-00005d6c0d23"
           (reference "R?") (unit 1)
@@
     (pin "2")
     (instances
-      (project "Incrementor"
+      (project "Stopwatch"
         (path "/c0d2575b-aec2-49ed-8c32-97fe6e68824c/00000000-0000-0000-0000-00005d6c0d23"
           (reference "R?") (unit 1)
@@
     (pin "1")
     (instances
-      (project "Incrementor"
+      (project "Stopwatch"
         (path "/c0d2575b-aec2-49ed-8c32-97fe6e68824c/00000000-0000-0000-0000-00005d77a516"
           (reference "TP203") (unit 1)
@@
     (pin "1")
     (instances
-      (project "Incrementor"
+      (project "Stopwatch"
         (path "/c0d2575b-aec2-49ed-8c32-97fe6e68824c/00000000-0000-0000-0000-00005d77a516"
           (reference "TP202") (unit 1)
@@
     (pin "1")
     (instances
-      (project "Incrementor"
+      (project "Stopwatch"
         (path "/c0d2575b-aec2-49ed-8c32-97fe6e68824c/00000000-0000-0000-0000-00005d77a516"
           (reference "TP201") (unit 1)
@@
     )
     (pin "1")
+    (instances
+      (project "Stopwatch"
+        (path "/c0d2575b-aec2-49ed-8c32-97fe6e68824c/00000000-0000-0000-0000-00005d77a516"
+          (reference "#PWR0203") (unit 1)
+        )
+      )
+    )
   )
   (symbol (lib_id "Custom_Library:C_Custom") (at 116.84 111.252 0) (unit 1)
     (in_bom yes) (on_board yes) (dnp no)
-    (property "Reference" "C?" (at 117.475 108.712 0)
+    (property "Reference" "C204" (at 117.475 108.712 0)
       (effects (font (size 1.27 1.27)) (justify left))
     )
@@
     (pin "2")
     (instances
-      (project "Incrementor"
+      (project "Stopwatch"
         (path "/c0d2575b-aec2-49ed-8c32-97fe6e68824c/00000000-0000-0000-0000-00005d77a516"
           (reference "C204") (unit 1)
@@
       (effects (font (size 1.27 1.27)) hide)
     )
-  )
+    (instances
+      (project "Stopwatch"
+        (path "/c0d2575b-aec2-49ed-8c32-97fe6e68824c/00000000-0000-0000-0000-00005d77a516"
+          (reference "N201") (unit 1)
+        )
+      )
+    )
+  )
