File: hdw/Incrementor/Pushbuttons.kicad_sch (KiCad schematic)
At the start: 41 parts, among them SW701 Cap_Touch, SW702 Cap_Touch, SW703 Cap_Touch, U701 AT42QT1010-TSHR, U702 TLV71330PDBV, U703 TLV71330PDBV, U704 74LVC1G80, U705 74LVC1G17, U706 TLV71330PDBV, U707 AT42QT1010-TSHR, U708 AT42QT1010-TSHR, U709 74LVC1G17, U710 74LVC1G17

Commit message: renamed project, removed stuff I dont need
Other:
- title: Incrementor -> Stopwatch
