File: hdw/Incrementor/Stage_01.kicad_sch (KiCad schematic)
At the start: 5 parts, among them U901 4026, U902 HDSP-7503

Commit message: renamed project, removed stuff I dont need
Other:
- title: Incrementor -> Stopwatch
Changed lines of the file:
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@@
   (paper "A")
   (title_block
-    (title "Incrementor")
-    (date "2019-09-03")
+    (title "Stopwatch")
+    (date "2024-01-02")
     (rev "A")
     (company "Drew Maatman")
@@
     (pin "9")
     (instances
-      (project "Incrementor"
+      (project "Stopwatch"
         (path "/c0d2575b-aec2-49ed-8c32-97fe6e68824c/00000000-0000-0000-0000-00005d6b2673"
           (reference "U901") (unit 1)
@@
     )
     (pin "1")
+    (instances
+      (project "Stopwatch"
+        (path "/c0d2575b-aec2-49ed-8c32-97fe6e68824c/00000000-0000-0000-0000-00005d6b2673"
+          (reference "#PWR0904") (unit 1)
+        )
+      )
+    )
   )
   (symbol (lib_id "power:GND") (at 118.872 112.268 0) (unit 1)
@@
     )
     (pin "1")
+    (instances
+      (project "Stopwatch"
+        (path "/c0d2575b-aec2-49ed-8c32-97fe6e68824c/00000000-0000-0000-0000-00005d6b2673"
+          (reference "#PWR0905") (unit 1)
+        )
+      )
+    )
   )
   (symbol (lib_id "Device:R_Pack08") (at 185.674 83.566 270) (unit 1)
@@
     (pin "9")
     (instances
-      (project "Incrementor"
+      (project "Stopwatch"
         (path "/c0d2575b-aec2-49ed-8c32-97fe6e68824c/00000000-0000-0000-0000-00005d6b2673"
           (reference "RN901") (unit 1)
@@
     (pin "9")
     (instances
-      (project "Incrementor"
+      (project "Stopwatch"
         (path "/c0d2575b-aec2-49ed-8c32-97fe6e68824c/00000000-0000-0000-0000-00005d6b2673"
           (reference "U902") (unit 1)
@@
     )
     (pin "1")
+    (instances
+      (project "Stopwatch"
+        (path "/c0d2575b-aec2-49ed-8c32-97fe6e68824c/00000000-0000-0000-0000-00005d6b2673"
+          (reference "#PWR0908") (unit 1)
+        )
+      )
+    )
   )
   (symbol (lib_id "Custom_Library:R_Custom") (at 76.2 112.014 0) (unit 1)
@@
     (pin "2")
     (instances
-      (project "Incrementor"
+      (project "Stopwatch"
         (path "/c0d2575b-aec2-49ed-8c32-97fe6e68824c/00000000-0000-0000-0000-00005d6b2673"
           (reference "R901") (unit 1)
@@
     )
     (pin "1")
+    (instances
+      (project "Stopwatch"
+        (path "/c0d2575b-aec2-49ed-8c32-97fe6e68824c/00000000-0000-0000-0000-00005d6b2673"
+          (reference "#PWR0901") (unit 1)
+        )
+      )
+    )
   )
   (symbol (lib_id "Custom_Library:C_Custom") (at 144.018 129.032 0) (unit 1)
@@
     (pin "2")
     (instances
-      (project "Incrementor"
+      (project "Stopwatch"
         (path "/c0d2575b-aec2-49ed-8c32-97fe6e68824c/00000000-0000-0000-0000-00005d6b2673"
           (reference "C901") (unit 1)
@@
     )
     (pin "1")
+    (instances
+      (project "Stopwatch"
+        (path "/c0d2575b-aec2-49ed-8c32-97fe6e68824c/00000000-0000-0000-0000-00005d6b2673"
+          (reference "#PWR0907") (unit 1)
+        )
+      )
+    )
   )
   (symbol (lib_id "Incrementor-rescue:+3.3V-power") (at 144.018 125.222 0) (unit 1)
@@
     )
     (pin "1")
+    (instances
+      (project "Stopwatch"
+        (path "/c0d2575b-aec2-49ed-8c32-97fe6e68824c/00000000-0000-0000-0000-00005d6b2673"
+          (reference "#PWR0906") (unit 1)
+        )
+      )
+    )
   )
 )
