File: hdw/Incrementor/Stage_03.kicad_sch (KiCad schematic)
At the start: 5 parts, among them U1101 4026, U1102 HDSP-7503

Commit message: renamed project, removed stuff I dont need
Other:
- title: Incrementor -> Stopwatch
Changed lines of the file:
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@@
   (paper "A")
   (title_block
-    (title "Incrementor")
-    (date "2019-09-03")
+    (title "Stopwatch")
+    (date "2024-01-02")
     (rev "A")
     (company "Drew Maatman")
@@
     (pin "9")
     (instances
-      (project "Incrementor"
+      (project "Stopwatch"
         (path "/c0d2575b-aec2-49ed-8c32-97fe6e68824c/00000000-0000-0000-0000-00005d6c0d1d"
           (reference "U1101") (unit 1)
@@
     (pin "1")
     (instances
-      (project "Incrementor"
+      (project "Stopwatch"
         (path "/c0d2575b-aec2-49ed-8c32-97fe6e68824c/00000000-0000-0000-0000-00005d6c0d1d"
           (reference "#PWR01104") (unit 1)
@@
     (pin "1")
     (instances
-      (project "Incrementor"
+      (project "Stopwatch"
         (path "/c0d2575b-aec2-49ed-8c32-97fe6e68824c/00000000-0000-0000-0000-00005d6c0d1d"
           (reference "#PWR01105") (unit 1)
@@
     (pin "9")
     (instances
-      (project "Incrementor"
+      (project "Stopwatch"
         (path "/c0d2575b-aec2-49ed-8c32-97fe6e68824c/00000000-0000-0000-0000-00005d6c0d1d"
           (reference "RN1101") (unit 1)
@@
     (pin "9")
     (instances
-      (project "Incrementor"
+      (project "Stopwatch"
         (path "/c0d2575b-aec2-49ed-8c32-97fe6e68824c/00000000-0000-0000-0000-00005d6c0d1d"
           (reference "U1102") (unit 1)
@@
     (pin "1")
     (instances
-      (project "Incrementor"
+      (project "Stopwatch"
         (path "/c0d2575b-aec2-49ed-8c32-97fe6e68824c/00000000-0000-0000-0000-00005d6c0d1d"
           (reference "#PWR01108") (unit 1)
@@
     (pin "2")
     (instances
-      (project "Incrementor"
+      (project "Stopwatch"
         (path "/c0d2575b-aec2-49ed-8c32-97fe6e68824c/00000000-0000-0000-0000-00005d6c0d1d"
           (reference "R1101") (unit 1)
@@
     (pin "1")
     (instances
-      (project "Incrementor"
+      (project "Stopwatch"
         (path "/c0d2575b-aec2-49ed-8c32-97fe6e68824c/00000000-0000-0000-0000-00005d6c0d1d"
           (reference "#PWR01101") (unit 1)
@@
     (pin "2")
     (instances
-      (project "Incrementor"
+      (project "Stopwatch"
         (path "/c0d2575b-aec2-49ed-8c32-97fe6e68824c/00000000-0000-0000-0000-00005d6c0d1d"
           (reference "C1101") (unit 1)
@@
     (pin "1")
     (instances
-      (project "Incrementor"
+      (project "Stopwatch"
         (path "/c0d2575b-aec2-49ed-8c32-97fe6e68824c/00000000-0000-0000-0000-00005d6c0d1d"
           (reference "#PWR01107") (unit 1)
@@
     (pin "1")
     (instances
-      (project "Incrementor"
+      (project "Stopwatch"
         (path "/c0d2575b-aec2-49ed-8c32-97fe6e68824c/00000000-0000-0000-0000-00005d6c0d1d"
           (reference "#PWR01106") (unit 1)
