File: hdw/Incrementor/Stage_09.kicad_sch (KiCad schematic)
At the start: 5 parts, among them U1701 4026, U1702 HDSP-7503

Commit message: renamed project, removed stuff I dont need
Other:
- title: Incrementor -> Stopwatch
Changed lines of the file:
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@@
   (paper "A")
   (title_block
-    (title "Incrementor")
-    (date "2019-09-03")
+    (title "Stopwatch")
+    (date "2024-01-02")
     (rev "A")
     (company "Drew Maatman")
