File: hdw/Incrementor/Status_LEDs.kicad_sch (KiCad schematic)
At the start: 43 parts, among them U601 74LVC1G06, U602 74LVC1G06, U603 74LVC1G06, U604 74LVC1G06, U605 74LVC1G06, U606 74LVC1G06, U607 74LVC1G06, U608 74LVC1G06, U609 74LVC1G06

Commit message: renamed project, removed stuff I dont need
Other:
- title: Incrementor -> Stopwatch
